File: hardware/kicad/SIM108.kicad_pcb (KiCad board)
At the start: 2 copper layers, 100 x 85 mm, 93 parts, among them J1 Screw_Terminal_01x09, J2 CAN, Q1 BC547, Q10 BC337, Q11 BC547, Q12 BC337, Q13 BC547, Q14 BC337, Q15 BC547, Q16 BC337, Q2 BC337, Q3 BC547, Q4 BC337, Q5 BC547, Q6 BC337, Q7 BC547, Q8 BC337, Q9 BC547, SW1 PRG, SW2 INSTANCE, SW3 BUS, U1 MCP2551-I-P, U10 SFH617A-1, U11 SFH617A-1, U12 SFH617A-1, U13 SFH617A-1, U14 MAX6816, U15 MAX6816, U16 MAX6816, U17 MAX6816, U18 MAX6816, U19 MAX6816, U2 TMR_2411, U20 MAX6816, U21 MAX6816, U3 MAX6816, U4 74HC595, U5 Teensy_3.2, U6 SFH617A-1, U7 SFH617A-1, U8 SFH617A-1, U9 SFH617A-1

Commit message: Layout
Parts:
- added C10: CP_Small, Capacitor_SMD:CP_Elec_4x4.5, F.Cu at (40.6, 84.5)
- added C11: CP_Small, Capacitor_SMD:CP_Elec_4x4.5, F.Cu at (50.7, 84.5)
- added C12: CP_Small, Capacitor_SMD:CP_Elec_4x4.5, F.Cu at (60.9, 84.5)
- added C5: CP_Small, Capacitor_SMD:CP_Elec_4x4.5, F.Cu at (-10.2, 84.5)
- added C6: CP_Small, Capacitor_SMD:CP_Elec_4x4.5, F.Cu at (-0.08, 84.5)
- added C7: CP_Small, Capacitor_SMD:CP_Elec_4x4.5, F.Cu at (10.1, 84.5)
- added C8: CP_Small, Capacitor_SMD:CP_Elec_4x4.5, F.Cu at (30.4, 84.5)
- added C9: CP_Small, Capacitor_SMD:CP_Elec_4x4.5, F.Cu at (20.2, 84.5)
- R19, R20, R21, R22, R23, R24, R25, R26: value 10K -> 100R; footprint Resistor_THT:R_Axial_DIN0207_L6.3mm_D2.5mm_P2.54mm_Vertical -> Resistor_SMD:R_0603_1608Metric_Pad0.98x0.95mm_HandSolder
- moved R26 61.4 mm to (5.38, 82.8), turned to 0 degrees
- moved R23 10.3 mm to (46.2, 83.4)
- moved R20 10.3 mm to (15.7, 83.4)
- moved R21 10.3 mm to (25.8, 83.4)
- moved R22 10.3 mm to (36.0, 83.4)
- moved R24 10.3 mm to (56.3, 83.4)
- moved R25 10.3 mm to (66.5, 83.4)
- moved U14 5.47 mm to (-4.78, 85.7), turned to 270 degrees
- moved U15 5.47 mm to (5.38, 85.7), turned to 270 degrees
- moved U16 5.21 mm to (15.3, 86.1)
- moved U17 5.21 mm to (25.5, 86.1)
- moved U19 5.21 mm to (45.8, 86.1)
- moved U20 5.21 mm to (55.9, 86.1)
- moved U18 5.21 mm to (35.6, 86.1)
- moved U21 5.21 mm to (66.1, 86.1)
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Connections:
- R19 pad 1: +5V -> Net-(R19-Pad1)
- R19 pad 2: Net-(R19-Pad2) -> GND
- R20 pad 1: +5V -> Net-(R20-Pad1)
- R20 pad 2: Net-(R20-Pad2) -> GND
- R21 pad 1: +5V -> Net-(R21-Pad1)
- R21 pad 2: Net-(R21-Pad2) -> GND
- R22 pad 1: +5V -> Net-(R22-Pad1)
- R22 pad 2: Net-(R22-Pad2) -> GND
- R23 pad 1: +5V -> Net-(R23-Pad1)
- R23 pad 2: Net-(R23-Pad2) -> GND
- R24 pad 1: +5V -> Net-(R24-Pad1)
- R24 pad 2: Net-(R24-Pad2) -> GND
- R25 pad 1: +5V -> Net-(R25-Pad1)
- R25 pad 2: Net-(R25-Pad2) -> GND
- R26 pad 1: +5V -> Net-(R26-Pad1)
- R26 pad 2: Net-(R26-Pad2) -> GND
- U10 pad 3: GND -> Net-(R22-Pad1)
- U10 pad 4: Net-(R23-Pad2) -> +5V
- U11 pad 3: GND -> Net-(R23-Pad1)
- U11 pad 4: Net-(R24-Pad2) -> +5V
- U12 pad 3: GND -> Net-(R24-Pad1)
- U12 pad 4: Net-(R25-Pad2) -> +5V
- U13 pad 3: GND -> Net-(R25-Pad1)
- U13 pad 4: Net-(R26-Pad2) -> +5V
- U14 pad 2: Net-(R19-Pad2) -> Net-(R19-Pad1)
- U15 pad 2: Net-(R20-Pad2) -> Net-(R26-Pad1)
- U16 pad 2: Net-(R21-Pad2) -> Net-(R20-Pad1)
- U17 pad 2: Net-(R22-Pad2) -> Net-(R21-Pad1)
- U18 pad 2: Net-(R23-Pad2) -> Net-(R22-Pad1)
- U19 pad 2: Net-(R24-Pad2) -> Net-(R23-Pad1)
- U20 pad 2: Net-(R25-Pad2) -> Net-(R24-Pad1)
- U21 pad 2: Net-(R26-Pad2) -> Net-(R25-Pad1)
- U5 pad 18: /CH0 -> /CH7
- U5 pad 19: /CH1 -> /CH6
- U5 pad 20: /CH2 -> /CH5
- U5 pad 21: /CH3 -> /CH4
- U5 pad 22: /CH4 -> /CH3
- U5 pad 23: /CH5 -> /CH2
- U5 pad 24: /CH7 -> /CH1
- U5 pad 25: /CH6 -> /CH0
- U6 pad 3: GND -> Net-(R19-Pad1)
- U6 pad 4: Net-(R19-Pad2) -> +5V
- U7 pad 3: GND -> Net-(R26-Pad1)
- U7 pad 4: Net-(R20-Pad2) -> +5V
- U8 pad 3: GND -> Net-(R20-Pad1)
- U8 pad 4: Net-(R21-Pad2) -> +5V
- U9 pad 3: GND -> Net-(R21-Pad1)
- U9 pad 4: Net-(R22-Pad2) -> +5V
Routing:
- net +5V: track 369.1 -> 436.7 mm
- net /CH0: track 102.9 -> 73.4 mm
- net /CH1: track 88.5 -> 66.3 mm
- net /CH7: track 43.8 -> 62.2 mm
- net /CH6: track 32.2 -> 49.4 mm
- net /CH2: track 74.1 -> 57.8 mm
- net Net-(R26-Pad1): track 0.00 -> 12.4 mm
- net Net-(R19-Pad1): track 0.00 -> 12.0 mm
- net Net-(R21-Pad1): track 0.00 -> 9.98 mm
- net Net-(R23-Pad1): track 0.00 -> 9.97 mm
- net Net-(R20-Pad1): track 0.00 -> 9.96 mm
- net Net-(R24-Pad1): track 0.00 -> 9.96 mm
- net Net-(R22-Pad1): track 0.00 -> 9.96 mm
- net Net-(R25-Pad1): track 0.00 -> 9.96 mm
- net /CH5: track 31.2 -> 39.5 mm
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
Commit message: Layout
Parts:
- moved R19 7.57 mm to (-11.0, 87.1)
- moved U14 5.98 mm to (-10.6, 84.5), turned to 0 degrees
- moved C5 4.19 mm to (-6.04, 84.5), turned to 270 degrees
- moved R20 0.65 mm to (15.5, 82.8), turned to 0 degrees
- moved U16 0.46 mm to (15.5, 85.7), turned to 270 degrees
Routing:
- net +5V: track 436.7 -> 426.2 mm
- net /CH2: track 57.8 -> 60.5 mm
- net Net-(R20-Pad1): track 9.96 -> 12.4 mm
- net /CH0: track 73.4 -> 72.6 mm
- net GND: track 10.8 -> 11.2 mm, vias 31 -> 33

Commit message: PCB layout
Parts:
- moved R20 7.57 mm to (9.32, 87.1)
- moved R26 7.57 mm to (-0.84, 87.1)
- moved R23 7.35 mm to (39.8, 87.1), turned to 0 degrees
- moved R21 7.34 mm to (19.5, 87.1), turned to 0 degrees
- moved R22 7.34 mm to (29.6, 87.1), turned to 0 degrees
- moved R24 7.34 mm to (50.0, 87.1), turned to 0 degrees
- moved R25 7.34 mm to (60.1, 87.1), turned to 0 degrees
- moved U16 5.98 mm to (9.70, 84.5), turned to 0 degrees
- moved U15 5.98 mm to (-0.46, 84.5), turned to 0 degrees
- moved U17 5.83 mm to (19.9, 84.5), turned to 0 degrees
- moved U19 5.83 mm to (40.2, 84.5), turned to 0 degrees
- moved U18 5.83 mm to (30.0, 84.5), turned to 0 degrees
- moved U20 5.83 mm to (50.3, 84.5), turned to 0 degrees
- moved U21 5.83 mm to (60.5, 84.5), turned to 0 degrees
- moved C10 4.19 mm to (44.8, 84.5), turned to 270 degrees
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Routing:
- net GND: track 11.2 -> 7.12 mm, vias 33 -> 53
- net /CH3: track 53.0 -> 55.3 mm
- net /CH4: track 45.9 -> 48.0 mm
- net +5V: track 426.2 -> 424.3 mm
- net Net-(R25-Pad1): track 9.96 -> 11.7 mm
- net Net-(R24-Pad1): track 9.96 -> 11.7 mm
- net Net-(R22-Pad1): track 9.96 -> 11.7 mm
- net Net-(R23-Pad1): track 9.97 -> 11.7 mm
- net Net-(R21-Pad1): track 9.98 -> 11.7 mm
- net /CH5: track 39.5 -> 41.3 mm
- net /CH1: track 66.3 -> 65.4 mm
- net Net-(R26-Pad1): track 12.4 -> 11.7 mm
- net Net-(R20-Pad1): track 12.4 -> 11.7 mm
- net /CH2: track 60.5 -> 59.9 mm
