File: hardware/kicad/SIM108.kicad_pcb (KiCad board)
At the start: 2 copper layers, 100 x 85 mm, 114 parts, among them J1 Screw_Terminal_01x09, J2 CAN, Q1 BC547, Q10 BC337-40, Q11 BC547, Q12 BC337-40, Q13 BC547, Q14 BC337-40, Q15 BC547, Q16 BC337-40, Q2 BC337-40, Q3 BC547, Q4 BC337-40, Q5 BC547, Q6 BC337-40, Q7 BC547, Q8 BC337-40, Q9 BC547, SW1 PRG, SW2 INSTANCE, SW3 BUS, U1 MCP2551-I-P, U10 SFH617A-1, U11 MAX6816, U12 SFH617A-1, U13 MAX6816, U14 SFH617A-1, U15 MAX6816, U16 SFH617A-1, U17 MAX6816, U18 SFH617A-1, U19 MAX6816, U2 TMR_2411, U20 SFH617A-1, U21 MAX6816, U3 MAX6816, U4 74HC595, U5 Teensy_3.2, U6 SFH617A-1, U7 MAX6816, U8 SFH617A-1, U9 MAX6816

Commit message: Refactor
Parts:
- U2: footprint PDJR-connectors:TMR_2411 -> PDJR_DC-DC_Converters:TMR_2411

Commit message: Refactor
Parts:
- J1: footprint PDJR-connectors:CAMDEN_BOSS_CSTBV2-9_TERMINAL -> PDJR_Connectors:CAMDEN_BOSS_CSTBV2-9_TERMINAL
- SW1: footprint PDJR-connectors:PCB_PUSH_BUTTON -> PDJR_Switches:PCB_PUSH_BUTTON_10mm
Other:
- board text added: "SIM108 NMEA 2000 Switch Input Module"
- board text removed: "SIM108 - NMEA 2000 Switch Input Module"

Commit message: Change relay terminal
Other:
- board text added: "SIM108 221101 (c) 2022 PDJR NMEA 2000 Switch Input Module"
- board text removed: "SIM108 NMEA 2000 Switch Input Module"

Commit message: Tweak
Parts:
- moved D16 36.9 mm to (96.6, 90.4)
- moved Q12 36.9 mm to (88.9, 84.7)
- moved Q14 36.9 mm to (98.9, 84.7)
- moved Q9 36.9 mm to (73.8, 84.7)
- moved R17 36.9 mm to (73.8, 81.6)
- moved R19 36.9 mm to (88.9, 81.6)
- moved R22 36.9 mm to (99.1, 81.6)
- moved C1 36.9 mm to (29.5, 43.7)
- moved D10 36.9 mm to (25.4, 90.4)
- moved D11 36.9 mm to (45.8, 90.4)
- moved D13 36.9 mm to (66.2, 90.4)
- moved D14 36.9 mm to (76.3, 90.4)
- moved D17 36.9 mm to (35.6, 90.4)
- moved D4 36.9 mm to (111.8, 53.2)
- moved D5 36.9 mm to (118.4, 53.2)
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Other:
- board text added: "CONNECT BUS SHIELD TO GROUND"
- board text added: "SIM108 221101 (c) 2022 PDJR/Paul Reeve NMEA 2000 Switch Input Module"
- board text added: "TERMINATE BUS (120R)"
- board text removed: "G"
- board text removed: "SIM108 221101 (c) 2022 PDJR NMEA 2000 Switch Input Module"
- board text removed: "T"

Commit message: PCB tweak
Other:
- board text added: "SIM108 Version 2211 NMEA 2000 Switch Input Module Copyright (c) 2022 PDJR"
- board text removed: "SIM108 221101 (c) 2022 PDJR/Paul Reeve NMEA 2000 Switch Input Module"
Changed lines of the file:
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@@
   (general
     (thickness 1.6)
-    (drawings 83)
+    (drawings 105)
     (tracks 974)
     (zones 0)
@@
     (0 F.Cu mixed)
     (31 B.Cu mixed)
-    (33 F.Adhes user)
+    (33 F.Adhes user hide)
     (35 F.Paste user)
     (37 F.SilkS user)
     (38 B.Mask user hide)
     (39 F.Mask user)
-    (40 Dwgs.User user)
+    (40 Dwgs.User user hide)
     (41 Cmts.User user hide)
     (42 Eco1.User user hide)
@@
     (aux_axis_origin 0 0)
     (grid_origin 100 0)
-    (visible_elements FFFFFF7F)
+    (visible_elements FFFFF77F)
     (pcbplotparams
       (layerselection 0x010e0_ffffffff)
@@
     )
   )
+  (gr_line (start 119.939 105.029) (end 119.939 60.96) (layer Dwgs.User) (width 0.15))
+  (gr_line (start 19.99 105.029) (end 119.939 105.029) (layer Dwgs.User) (width 0.15))
+  (gr_line (start 19.99 60.96) (end 19.99 105.029) (layer Dwgs.User) (width 0.15))
+  (gr_line (start 119.939 60.96) (end 19.99 60.96) (layer Dwgs.User) (width 0.15))
+  (gr_line (start 19.99 30.48) (end 19.99 20.066) (layer Dwgs.User) (width 0.15))
+  (gr_line (start 54.661 30.48) (end 19.99 30.48) (layer Dwgs.User) (width 0.15))
+  (gr_line (start 54.661 47.752) (end 54.661 30.861) (layer Dwgs.User) (width 0.15))
+  (gr_line (start 19.99 47.752) (end 54.661 47.752) (layer Dwgs.User) (width 0.15))
+  (gr_line (start 19.99 30.861) (end 19.99 47.752) (layer Dwgs.User) (width 0.15))
+  (gr_line (start 54.661 30.861) (end 19.99 30.861) (layer Dwgs.User) (width 0.15))
+  (gr_line (start 54.661 20.066) (end 54.661 30.48) (layer Dwgs.User) (width 0.15))
+  (gr_line (start 19.99 20.066) (end 54.661 20.066) (layer Dwgs.User) (width 0.15))
+  (gr_line (start 119.939 60.579) (end 90.094 60.579) (layer Dwgs.User) (width 0.15))
+  (gr_line (start 119.939 34.798) (end 119.939 60.579) (layer Dwgs.User) (width 0.15))
+  (gr_line (start 90.094 34.798) (end 119.939 34.798) (layer Dwgs.User) (width 0.15))
+  (gr_line (start 90.094 60.579) (end 90.094 34.798) (layer Dwgs.User) (width 0.15))
+  (gr_line (start 119.939 19.939) (end 55.042 20.066) (layer Dwgs.User) (width 0.15))
+  (gr_line (start 119.939 34.417) (end 119.939 19.939) (layer Dwgs.User) (width 0.15))
+  (gr_line (start 89.713 34.417) (end 119.939 34.417) (layer Dwgs.User) (width 0.15))
+  (gr_line (start 89.713 60.579) (end 89.713 34.417) (layer Dwgs.User) (width 0.15))
+  (gr_line (start 55.042 60.579) (end 89.713 60.579) (layer Dwgs.User) (width 0.15))
+  (gr_line (start 55.042 20.066) (end 55.042 60.579) (layer Dwgs.User) (width 0.15))
   (gr_text H (at 21.463 42.52) (layer F.SilkS)
     (effects (font (size 1 1) (thickness 0.15)))
@@
     (effects (font (size 1 1) (thickness 0.15)))
   )
-  (gr_text "SIM108 221101 (c) 2022 PDJR/Paul Reeve\nNMEA 2000 Switch Input Module\n" (at 21 52) (layer F.SilkS)
+  (gr_text "SIM108 Version 2211\nNMEA 2000 Switch Input Module\nCopyright (c) 2022 PDJR" (at 21 55) (layer F.SilkS)
     (effects (font (size 2 1.5) (thickness 0.3)) (justify left))
   )
@@
     (connect_pads (clearance 0.508))
     (min_thickness 0.254)
-    (fill (arc_segments 32) (thermal_gap 0.508) (thermal_bridge_width 0.508))
+    (fill yes (arc_segments 32) (thermal_gap 0.508) (thermal_bridge_width 0.508))
     (polygon
       (pts
@@
     (connect_pads (clearance 0.508))
     (min_thickness 0.254)
-    (fill (arc_segments 32) (thermal_gap 0.508) (thermal_bridge_width 0.508))
+    (fill yes (arc_segments 32) (thermal_gap 0.508) (thermal_bridge_width 0.508))
     (polygon
       (pts

Commit message: PCB tweak
Other:
- board text added: "BEFORE USE assign this module a unique instance address by setting ‘INSTANCE’ to the required value and pressing ‘PRG’. The assigned value must not be in use by another switchbank on the same NMEA network and must be in the range 0..252. MAKE SURE that the settings of ‘CONNECT BUS SHIELD TO GROUND’ and ‘TERMINATE BUS (120R)’ reflect your installation choices."
