File: hardware/kicad/SIM108.sch (KiCad schematic (older format))
At the start: 33 parts, among them J1 Screw_Terminal_01x09, J2 CAN, SW1 INSTANCE, SW2 BUS, U1 74HC595, U2 MCP2551-I-P, U3 TMR-1211, U4 Teensy_3.2

Commit message: New board size
Parts:
- removed C1: 100nF, Capacitor_THT:C_Rect_L4.6mm_W2.0mm_P2.50mm_MKS02_FKP02, symbol Device:C
- removed C2: 100n, Capacitor_THT:C_Rect_L4.6mm_W3.0mm_P2.50mm_MKS02_FKP02, symbol Device:C
- removed C3: 1000uF, Capacitor_THT:CP_Radial_D8.0mm_P5.00mm, symbol Device:CP
- removed D1, D2, D3, D4, D5, D6, D7, D8, D9: LED_Small, LED_THT:LED_Rectangular_W3.0mm_H2.0mm, symbol Device:LED_Small
- removed R1, R3, R4, R5, R6, R7, R8: 470R, Resistor_THT:R_Axial_DIN0207_L6.3mm_D2.5mm_P2.54mm_Vertical, symbol Device:R
- removed R11: 120R, Resistor_THT:R_Axial_DIN0207_L6.3mm_D2.5mm_P7.62mm_Horizontal, symbol Device:R
- removed R9: 470R, Resistor_THT:R_Axial_DIN0207_L6.3mm_D2.5mm_P7.62mm_Horizontal, symbol Device:R
- removed SW1: INSTANCE, Package_DIP:DIP-16_W7.62mm, symbol Switch:SW_DIP_x08
- removed U1: 74HC595, Package_DIP:DIP-16_W7.62mm, symbol 74xx:74HC595
- removed U3: TMR-1211, PDJR-connectors:TMR-1-1211, symbol pdjr:TMR-1211
- added C1, C2, C4: 100nF, Capacitor_THT:CP_Radial_D5.0mm_P2.00mm, symbol Device:CP_Small
- added D1, D2, D3, D4, D5, D6, D7, D8: LED, LED_THT:LED_D1.8mm_W3.3mm_H2.4mm, symbol Device:LED
- added RN1: R_Network08, Resistor_THT:R_Array_SIP9, symbol Device:R_Network08
- added SW1: PRG, PDJR-connectors:PCB_PUSH_BUTTON, symbol Switch:SW_Push
- added SW2: INSTANCE, Package_DIP:DIP-16_W7.62mm, symbol Switch:SW_DIP_x08
- added U2: TMR_2411, PDJR-connectors:TMR_2411, symbol pdjr:TMR_2411
- added U3: MAX6816, Package_TO_SOT_SMD:SOT-143, symbol Interface:MAX6816
- added U4: 74HC595, Package_DIP:DIP-16_W7.62mm_Socket_LongPads, symbol 74xx:74HC595
- C3: renamed from C4; footprint Capacitor_THT:C_Rect_L4.6mm_W3.0mm_P2.50mm_MKS02_FKP02 -> Capacitor_THT:CP_Radial_D5.0mm_P2.00mm
- J2: footprint TerminalBlock_Phoenix:TerminalBlock_Phoenix_MPT-0,5-5-2.54_1x05_P2.54mm_Horizontal -> Connector_PinHeader_2.54mm:PinHeader_1x05_P2.54mm_Vertical
- R2: value 470R -> 120R; footprint Resistor_THT:R_Axial_DIN0207_L6.3mm_D2.5mm_P2.54mm_Vertical -> Resistor_THT:R_Axial_DIN0207_L6.3mm_D2.5mm_P7.62mm_Horizontal; Power 0.125W -> (none)
- renumbered R10 to R1, SW2 to SW3, U2 to U1, U4 to U5
Connections:
- net labels added: MPX_CLOCK, MPX_DATA, MPX_LATCH, PRG
- net labels removed: CLOCK, DATA, LATCH, LED_PWR, NET_S
- wire segments 152 -> 167
Other:
- note added: "CONFIGURATION"
- note added: "DISPLAY"
- note added: "POWER SUPPLY & CAN INTERFACE"
- note removed: "12/5 V DC-DC CONVERTER"
- note removed: "CAN INTERFACE"
- note removed: "LED INDICATORS"
- moved on the sheet: C3, F1, J1, R1, SW3, U1, U5

Commit message: PCB tweak
Parts:
- U2: symbol pdjr:TMR_2411 -> SIM108-rescue:TMR_2411-pdjr
- U5: symbol pdjr:Teensy_3.2 -> SIM108-rescue:Teensy_3.2-pdjr
Changed lines of the file:
@@
 	9050 2900 9050 3250
 $Comp
-L pdjr:Teensy_3.2 U5
+L SIM108-rescue:Teensy_3.2-pdjr U5
 U 1 1 60F2AB82
 P 10250 2900
@@
 $EndComp
 $Comp
-L pdjr:TMR_2411 U2
+L SIM108-rescue:TMR_2411-pdjr U2
 U 1 1 6327DB22
 P 2900 5150

Commit message: Stuff
Connections:
- net CH0: now also U5.18 (D16); no longer U5.25 (D23)
- net CH7: now also U5.25 (D23); no longer U5.18 (D16)
Changed lines of the file:
@@
 NoConn ~ 9600 1400
 NoConn ~ 9500 1400
-Text Label 9150 2600 2    50   ~ 0
+Text Label 9150 1900 2    50   ~ 0
 CH0
 Text Label 9150 2500 2    50   ~ 0
@@
 Text Label 9150 2000 2    50   ~ 0
 CH6
-Text Label 9150 1900 2    50   ~ 0
+Text Label 9150 2600 2    50   ~ 0
 CH7
 $Comp
@@
 Opto-isolated SPST inputs. Each opto-isolator\nis driven by a constant current source which\noperates the isolator LED at 6mA from voltages\nin the range 5VDC through 50VDC.
 $Sheet
-S 3750 700  1100 300
+S 3750 700  1100 400
 U 62FB7846
 F0 "OII_00" 50
 F1 "opto_isolated_input.sch" 50
-F2 "OII_IN" I L 3750 800 50
-F3 "OII_IN_GND" U L 3750 900 50
-F4 "OII_OUT" O R 4850 800 50
-F5 "OII_OUT_GND" U R 4850 900 50
+F2 "OII_IN" I L 3750 900 50
+F3 "OII_IN_GND" U L 3750 1000 50
+F4 "OII_OUT" O R 4850 900 50
+F5 "OII_OUT_GND" U R 4850 1000 50
+F6 "OII_OUT_VCC" I R 4850 800 50
 $EndSheet
-Text Label 3650 800  2    50   ~ 0
+Text Label 3650 900  2    50   ~ 0
 SPST_CH0
-Text Label 3650 900  2    50   ~ 0
+Text Label 3650 1000 2    50   ~ 0
 SPST_GND
-Text Label 4950 800  0    50   ~ 0
+Text Label 4950 900  0    50   ~ 0
 CH0
 $Comp
@@
 $EndComp
 Wire Wire Line
-	4850 900  4950 900
-Wire Wire Line
-	4950 900  4950 1000
+	4850 1000 4950 1000
 Wire Wire Line
 	4950 800  4850 800
 Wire Wire Line
-	3650 800  3750 800
+	3650 1000 3750 1000
 Wire Wire Line
 	3650 900  3750 900
@@
 NoConn ~ 9150 1600
 NoConn ~ -3250 8100
+Wire Wire Line
+	4850 900  4950 900
+$Comp
+L power:+5V #PWR020
+U 1 1 634AE8DC
+P 4950 800
+F 0 "#PWR020" H 4950 650 50  0001 C CNN
+F 1 "+5V" H 4965 973 50  0000 C CNN
+F 2 "" H 4950 800 50  0001 C CNN
+F 3 "" H 4950 800 50  0001 C CNN
+	1    4950 800
+	1    0    0    -1
+$EndComp
 $EndSCHEMATC

Commit message: Debounce
Connections:
- net CH1: now also U5.19 (D17); no longer U5.24 (D22)
- net CH2: now also U5.20 (D18); no longer U5.23 (D21)
- net CH3: now also U5.21 (D19); no longer U5.22 (D20)
- net CH4: now also U5.22 (D20); no longer U5.21 (D19)
- net CH5: now also U5.23 (D21); no longer U5.20 (D18)
- net CH6: now also U5.25 (D23); no longer U5.19 (D17)
- net CH7: now also U5.24 (D22); no longer U5.25 (D23)
Changed lines of the file:
@@
 Text Label 9150 1900 2    50   ~ 0
 CH0
+Text Label 9150 2000 2    50   ~ 0
+CH1
+Text Label 9150 2100 2    50   ~ 0
+CH2
+Text Label 9150 2200 2    50   ~ 0
+CH3
+Text Label 9150 2300 2    50   ~ 0
+CH4
+Text Label 9150 2400 2    50   ~ 0
+CH5
+Text Label 9150 2600 2    50   ~ 0
+CH6
 Text Label 9150 2500 2    50   ~ 0
-CH1
-Text Label 9150 2400 2    50   ~ 0
-CH2
-Text Label 9150 2300 2    50   ~ 0
-CH3
-Text Label 9150 2200 2    50   ~ 0
-CH4
-Text Label 9150 2100 2    50   ~ 0
-CH5
-Text Label 9150 2000 2    50   ~ 0
-CH6
-Text Label 9150 2600 2    50   ~ 0
 CH7
 $Comp
@@
 Wire Wire Line
 	3650 900  3750 900
-$Sheet
-S 3750 1350 1100 300
-U 63089671
-F0 "OII_01" 50
-F1 "opto_isolated_input.sch" 50
-F2 "OII_IN" I L 3750 1450 50
-F3 "OII_IN_GND" U L 3750 1550 50
-F4 "OII_OUT" O R 4850 1450 50
-F5 "OII_OUT_GND" U R 4850 1550 50
-$EndSheet
-Wire Wire Line
-	4850 1450 4950 1450
-Wire Wire Line
-	4850 1550 4950 1550
-Wire Wire Line
-	4950 1550 4950 1650
-Wire Wire Line
-	3750 1450 3650 1450
-Wire Wire Line
-	3750 1550 3650 1550
-Text Label 3650 1450 2    50   ~ 0
+Text Label 3650 1550 2    50   ~ 0
 SPST_CH1
-Text Label 3650 1550 2    50   ~ 0
+Text Label 3650 1650 2    50   ~ 0
 SPST_GND
-Text Label 4950 1450 0    50   ~ 0
+Text Label 4950 1550 0    50   ~ 0
 CH1
 $Comp
@@
 $EndComp
 $Sheet
-S 3750 2000 1100 300
+S 3750 2000 1100 400
 U 63103CAF
 F0 "OII_02" 50
 F1 "opto_isolated_input.sch" 50
-F2 "OII_IN" I L 3750 2100 50
-F3 "OII_IN_GND" U L 3750 2200 50
-F4 "OII_OUT" O R 4850 2100 50
-F5 "OII_OUT_GND" U R 4850 2200 50
+F2 "OII_IN" I L 3750 2200 50
+F3 "OII_IN_GND" U L 3750 2300 50
+F4 "OII_OUT" O R 4850 2200 50
+F5 "OII_OUT_GND" U R 4850 2300 50
+F6 "OII_OUT_VCC" I R 4850 2100 50
 $EndSheet
 Wire Wire Line
-	4850 2100 4950 2100
-Wire Wire Line
-	4850 2200 4950 2200
-Wire Wire Line
-	4950 2200 4950 2300
-Wire Wire Line
-	3750 2100 3650 2100
+	4850 2300 4950 2300
+Wire Wire Line
+	3750 2300 3650 2300
 Wire Wire Line
 	3750 2200 3650 2200
-Text Label 3650 2100 2    50   ~ 0
+Text Label 3650 2200 2    50   ~ 0
 SPST_CH2
-Text Label 3650 2200 2    50   ~ 0
+Text Label 3650 2300 2    50   ~ 0
 SPST_GND
-Text Label 4950 2100 0    50   ~ 0
+Text Label 4950 2200 0    50   ~ 0
 CH2
 $Comp
@@
 $EndComp
 $Sheet
-S 3750 2650 1100 300
+S 3750 2650 1100 400
 U 62F64647
 F0 "OOI_03" 50
 F1 "opto_isolated_input.sch" 50
-F2 "OII_IN" I L 3750 2750 50
-F3 "OII_IN_GND" U L 3750 2850 50
-F4 "OII_OUT" O R 4850 2750 50
-F5 "OII_OUT_GND" U R 4850 2850 50
+F2 "OII_IN" I L 3750 2850 50
+F3 "OII_IN_GND" U L 3750 2950 50
+F4 "OII_OUT" O R 4850 2850 50
+F5 "OII_OUT_GND" U R 4850 2950 50
+F6 "OII_OUT_VCC" I R 4850 2750 50
 $EndSheet
 Wire Wire Line
@@
 	4850 2850 4950 2850
 Wire Wire Line
-	3750 2750 3650 2750
-Wire Wire Line
 	3750 2850 3650 2850
-Text Label 4950 2750 0    50   ~ 0
+Text Label 4950 2850 0    50   ~ 0
 CH3
 $Comp
@@
 	1    0    0    -1
 $EndComp
-Text Label 3650 2750 2    50   ~ 0
+Text Label 3650 2850 2    50   ~ 0
 SPST_CH3
-Text Label 3650 2850 2    50   ~ 0
+Text Label 3650 2950 2    50   ~ 0
 SPST_GND
-Wire Wire Line
-	4950 2850 4950 2950
 $Sheet
-S 5750 700  1100 300
+S 5750 700  1100 400
 U 62FD589D
 F0 "OOI_04" 50
 F1 "opto_isolated_input.sch" 50
-F2 "OII_IN" I L 5750 800 50
-F3 "OII_IN_GND" U L 5750 900 50
-F4 "OII_OUT" O R 6850 800 50
-F5 "OII_OUT_GND" U R 6850 900 50
+F2 "OII_IN" I L 5750 900 50
+F3 "OII_IN_GND" U L 5750 1000 50
+F4 "OII_OUT" O R 6850 900 50
+F5 "OII_OUT_GND" U R 6850 1000 50
+F6 "OII_OUT_VCC" I R 6850 800 50
 $EndSheet
 Wire Wire Line
@@
 	6850 900  6950 900
 Wire Wire Line
-	6950 900  6950 1000
-Wire Wire Line
-	5750 800  5650 800
-Wire Wire Line
 	5750 900  5650 900
-Text Label 5650 800  2    50   ~ 0
+Text Label 5650 900  2    50   ~ 0
 SPST_CH4
-Text Label 5650 900  2    50   ~ 0
+Text Label 5650 1000 2    50   ~ 0
 SPST_GND
-Text Label 6950 800  0    50   ~ 0
+Text Label 6950 900  0    50   ~ 0
 CH4
 $Comp
@@
 $EndComp
 $Sheet
-S 5750 1350 1100 300
+S 5750 1350 1100 400
 U 63041ECA
 F0 "OOI_05" 50
 F1 "opto_isolated_input.sch" 50
-F2 "OII_IN" I L 5750 1450 50
-F3 "OII_IN_GND" U L 5750 1550 50
-F4 "OII_OUT" O R 6850 1450 50
-F5 "OII_OUT_GND" U R 6850 1550 50
+F2 "OII_IN" I L 5750 1550 50
+F3 "OII_IN_GND" U L 5750 1650 50
+F4 "OII_OUT" O R 6850 1550 50
+F5 "OII_OUT_GND" U R 6850 1650 50
+F6 "OII_OUT_VCC" I R 6850 1450 50
 $EndSheet
 Wire Wire Line
@@
 	6850 1550 6950 1550
 Wire Wire Line
-	6950 1550 6950 1650
-Wire Wire Line
-	5750 1450 5650 1450
-Wire Wire Line
 	5750 1550 5650 1550
-Text Label 5650 1450 2    50   ~ 0
+Text Label 5650 1550 2    50   ~ 0
 SPST_CH5
-Text Label 5650 1550 2    50   ~ 0
+Text Label 5650 1650 2    50   ~ 0
 SPST_GND
-Text Label 6950 1450 0    50   ~ 0
+Text Label 6950 1550 0    50   ~ 0
 CH5
 $Comp
@@
 $EndComp
 $Sheet
-S 5750 2000 1100 300
+S 5750 2000 1100 400
 U 62F45EE0
 F0 "OOI_06" 50
 F1 "opto_isolated_input.sch" 50
-F2 "OII_IN" I L 5750 2100 50
-F3 "OII_IN_GND" U L 5750 2200 50
-F4 "OII_OUT" O R 6850 2100 50
-F5 "OII_OUT_GND" U R 6850 2200 50
+F2 "OII_IN" I L 5750 2200 50
+F3 "OII_IN_GND" U L 5750 2300 50
+F4 "OII_OUT" O R 6850 2200 50
+F5 "OII_OUT_GND" U R 6850 2300 50
+F6 "OII_OUT_VCC" I R 6850 2100 50
 $EndSheet
 Wire Wire Line
-	5750 2100 5650 2100
-Wire Wire Line
 	5750 2200 5650 2200
 Wire Wire Line
@@
 Wire Wire Line
 	6850 2200 6950 2200
-Wire Wire Line
-	6950 2200 6950 2300
-Text Label 5650 2100 2    50   ~ 0
+Text Label 5650 2200 2    50   ~ 0
 SPST_CH6
-Text Label 5650 2200 2    50   ~ 0
+Text Label 5650 2300 2    50   ~ 0
 SPST_GND
-Text Label 6950 2100 0    50   ~ 0
+Text Label 6950 2200 0    50   ~ 0
 CH6
 $Comp
@@
 $EndComp
 $Sheet
-S 5750 2650 1100 300
+S 5750 2650 1100 400
 U 62FB890E
 F0 "OII_07" 50
 F1 "opto_isolated_input.sch" 50
-F2 "OII_IN" I L 5750 2750 50
-F3 "OII_IN_GND" U L 5750 2850 50
-F4 "OII_OUT" O R 6850 2750 50
-F5 "OII_OUT_GND" U R 6850 2850 50
+F2 "OII_IN" I L 5750 2850 50
+F3 "OII_IN_GND" U L 5750 2950 50
+F4 "OII_OUT" O R 6850 2850 50
+F5 "OII_OUT_GND" U R 6850 2950 50
+F6 "OII_OUT_VCC" I R 6850 2750 50
 $EndSheet
 Wire Wire Line
@@
 Wire Wire Line
 	6850 2850 6950 2850
-Wire Wire Line
-	6950 2850 6950 2950
-Wire Wire Line
-	5750 2750 5650 2750
 Wire Wire Line
 	5750 2850 5650 2850
@@
 	1    0    0    -1
 $EndComp
-Text Label 5650 2750 2    50   ~ 0
+Text Label 5650 2850 2    50   ~ 0
 SPST_CH7
-Text Label 5650 2850 2    50   ~ 0
-SPST_GND
-Text Label 6950 2750 0    50   ~ 0
+Text Label 6950 2850 0    50   ~ 0
 CH7
 $Comp
@@
 	1    0    0    -1
 $EndComp
+$Sheet
+S 3750 1350 1100 400
+U 63089671
+F0 "OII_01" 50
+F1 "opto_isolated_input.sch" 50
+F2 "OII_IN" I L 3750 1550 50
+F3 "OII_IN_GND" U L 3750 1650 50
+F4 "OII_OUT" O R 4850 1550 50
+F5 "OII_OUT_GND" U R 4850 1650 50
+F6 "OII_OUT_VCC" I R 4850 1450 50
+$EndSheet
+$Comp
+L power:+5V #PWR021
+U 1 1 63462A09
+P 4950 1450
+F 0 "#PWR021" H 4950 1300 50  0001 C CNN
+F 1 "+5V" H 4965 1623 50  0000 C CNN
+F 2 "" H 4950 1450 50  0001 C CNN
+F 3 "" H 4950 1450 50  0001 C CNN
+	1    4950 1450
+	1    0    0    -1
+$EndComp
+Wire Wire Line
+	3650 1550 3750 1550
+Wire Wire Line
+	3650 1650 3750 1650
+Wire Wire Line
+	4850 1450 4950 1450
+Wire Wire Line
+	4850 1550 4950 1550
+Wire Wire Line
+	4850 1650 4950 1650
+$Comp
+L power:+5V #PWR0101
+U 1 1 634E105F
+P 4950 2100
+F 0 "#PWR0101" H 4950 1950 50  0001 C CNN
+F 1 "+5V" H 4965 2273 50  0000 C CNN
+F 2 "" H 4950 2100 50  0001 C CNN
+F 3 "" H 4950 2100 50  0001 C CNN
+	1    4950 2100
+	1    0    0    -1
+$EndComp
+Wire Wire Line
+	4850 2100 4950 2100
+Wire Wire Line
+	4850 2200 4950 2200
+Wire Wire Line
+	4850 2950 4950 2950
+$Comp
+L power:+5V #PWR0102
+U 1 1 6351340F
+P 4950 2750
+F 0 "#PWR0102" H 4950 2600 50  0001 C CNN
+F 1 "+5V" H 4965 2923 50  0000 C CNN
+F 2 "" H 4950 2750 50  0001 C CNN
+F 3 "" H 4950 2750 50  0001 C CNN
+	1    4950 2750
+	1    0    0    -1
+$EndComp
+Wire Wire Line
+	3650 2950 3750 2950
+Wire Wire Line
+	6850 1000 6950 1000
+$Comp
+L power:+5V #PWR0103
+U 1 1 6352F708
+P 6950 800
+F 0 "#PWR0103" H 6950 650 50  0001 C CNN
+F 1 "+5V" H 6965 973 50  0000 C CNN
+F 2 "" H 6950 800 50  0001 C CNN
+F 3 "" H 6950 800 50  0001 C CNN
+	1    6950 800
+	1    0    0    -1
+$EndComp
+Wire Wire Line
+	5750 1000 5650 1000
+Wire Wire Line
+	6850 1650 6950 1650
+Wire Wire Line
+	6850 2300 6950 2300
+Wire Wire Line
+	6850 2950 6950 2950
+$Comp
+L power:+5V #PWR0104
+U 1 1 6359AF9F
+P 6950 1450
+F 0 "#PWR0104" H 6950 1300 50  0001 C CNN
+F 1 "+5V" H 6965 1623 50  0000 C CNN
+F 2 "" H 6950 1450 50  0001 C CNN
+F 3 "" H 6950 1450 50  0001 C CNN
+	1    6950 1450
+	1    0    0    -1
+$EndComp
+$Comp
+L power:+5V #PWR0105
+U 1 1 6359B793
+P 6950 2100
+F 0 "#PWR0105" H 6950 1950 50  0001 C CNN
+F 1 "+5V" H 6965 2273 50  0000 C CNN
+F 2 "" H 6950 2100 50  0001 C CNN
+F 3 "" H 6950 2100 50  0001 C CNN
+	1    6950 2100
+	1    0    0    -1
+$EndComp
+$Comp
+L power:+5V #PWR0106
+U 1 1 6359BE30
+P 6950 2750
+F 0 "#PWR0106" H 6950 2600 50  0001 C CNN
+F 1 "+5V" H 6965 2923 50  0000 C CNN
+F 2 "" H 6950 2750 50  0001 C CNN
+F 3 "" H 6950 2750 50  0001 C CNN
+	1    6950 2750
+	1    0    0    -1
+$EndComp
+Text Label 5650 2950 2    50   ~ 0
+SPST_GND
+Wire Wire Line
+	5650 2950 5750 2950
+Wire Wire Line
+	5750 2300 5650 2300
+Wire Wire Line
+	5750 1650 5650 1650
 $EndSCHEMATC

Commit message: Layout
Connections:
- net CH0: now also U5.25 (D23); no longer U5.18 (D16)
- net CH1: now also U5.24 (D22); no longer U5.19 (D17)
- net CH2: now also U5.23 (D21); no longer U5.20 (D18)
- net CH3: now also U5.22 (D20); no longer U5.21 (D19)
- net CH4: now also U5.21 (D19); no longer U5.22 (D20)
- net CH5: now also U5.20 (D18); no longer U5.23 (D21)
- net CH6: now also U5.19 (D17); no longer U5.25 (D23)
- net CH7: now also U5.18 (D16); no longer U5.24 (D22)
Changed lines of the file:
@@
 NoConn ~ 9600 1400
 NoConn ~ 9500 1400
+Text Label 9150 2600 2    50   ~ 0
+CH0
+Text Label 9150 2500 2    50   ~ 0
+CH1
+Text Label 9150 2400 2    50   ~ 0
+CH2
+Text Label 9150 2300 2    50   ~ 0
+CH3
+Text Label 9150 2200 2    50   ~ 0
+CH4
+Text Label 9150 2100 2    50   ~ 0
+CH5
+Text Label 9150 2000 2    50   ~ 0
+CH6
 Text Label 9150 1900 2    50   ~ 0
-CH0
-Text Label 9150 2000 2    50   ~ 0
-CH1
-Text Label 9150 2100 2    50   ~ 0
-CH2
-Text Label 9150 2200 2    50   ~ 0
-CH3
-Text Label 9150 2300 2    50   ~ 0
-CH4
-Text Label 9150 2400 2    50   ~ 0
-CH5
-Text Label 9150 2600 2    50   ~ 0
-CH6
-Text Label 9150 2500 2    50   ~ 0
 CH7
 $Comp

Commit message: Add transmit LED
Parts:
- added D17: LED, LED_THT:LED_D1.8mm_W3.3mm_H2.4mm, symbol Device:LED
- added R27: 4K7, Resistor_THT:R_Axial_DIN0207_L6.3mm_D2.5mm_P2.54mm_Vertical, symbol Device:R
Connections:
- net GND: now also R27.2
- net TRANSMIT_LED: now reaches U5.17 (D15)
- net TRANSMIT_LED: now also D17.2 (A)
- new net: D17.1 (K), R27.1
- no-connect marks 9 -> 8
Changed lines of the file:
@@
 Text Label 9150 1700 2    50   ~ 0
 PRG
-NoConn ~ 9150 1800
 NoConn ~ 9150 1600
 NoConn ~ -3250 8100
@@
 Wire Wire Line
 	5750 1650 5650 1650
+$Comp
+L Device:LED D17
+U 1 1 6348B352
+P 9850 4300
+F 0 "D17" H 9950 4250 50  0000 C CNN
+F 1 "LED" H 9843 4136 50  0001 C CNN
+F 2 "LED_THT:LED_D1.8mm_W3.3mm_H2.4mm" H 9850 4300 50  0001 C CNN
+F 3 "~" H 9850 4300 50  0001 C CNN
+	1    9850 4300
+	-1   0    0    1
+$EndComp
+$Comp
+L Device:R R27
+U 1 1 63493E4A
+P 10150 4300
+F 0 "R27" H 10100 4300 50  0000 R CNN
+F 1 "4K7" V 10150 4300 39  0000 C CNN
+F 2 "Resistor_THT:R_Axial_DIN0207_L6.3mm_D2.5mm_P2.54mm_Vertical" V 10080 4300 50  0001 C CNN
+F 3 "~" H 10150 4300 50  0001 C CNN
+	1    10150 4300
+	0    -1   -1   0
+$EndComp
+$Comp
+L power:GND #PWR0107
+U 1 1 63496532
+P 10400 4400
+F 0 "#PWR0107" H 10400 4150 50  0001 C CNN
+F 1 "GND" H 10405 4227 50  0000 C CNN
+F 2 "" H 10400 4400 50  0001 C CNN
+F 3 "" H 10400 4400 50  0001 C CNN
+	1    10400 4400
+	1    0    0    -1
+$EndComp
+Wire Wire Line
+	10300 4300 10400 4300
+Wire Wire Line
+	10400 4300 10400 4400
+Wire Wire Line
+	9700 4300 9600 4300
+Text Label 9600 4300 2    50   ~ 0
+TRANSMIT_LED
+Text Label 9150 1800 2    50   ~ 0
+TRANSMIT_LED
 $EndSCHEMATC

Commit message: Change PCB conn
Parts:
- removed C3: 100nF, Capacitor_THT:CP_Radial_D5.0mm_P2.00mm, symbol Device:C
- added C3: 100nF, Capacitor_THT:CP_Radial_D5.0mm_P2.00mm, symbol Device:CP_Small
- R1: value 4K7 -> 4K7 0.125W; footprint Resistor_THT:R_Axial_DIN0207_L6.3mm_D2.5mm_P7.62mm_Horizontal -> Resistor_THT:R_Axial_DIN0207_L6.3mm_D2.5mm_P2.54mm_Vertical
- R2: value 120R -> 120R 0.5W
- renumbered D17 to D5, D5 to D6, D6 to D7, D7 to D8, D8 to D9, R27 to R3
Connections:
- net +5V: now also C3.1
- net GND: now also C3.2

Commit message: Update connector
Parts:
- J1: footprint TerminalBlock_Phoenix:TerminalBlock_Phoenix_MKDS-3-9-5.08_1x09_P5.08mm_Horizontal -> PDJR-connectors:RS-PLUG-TERMINAL-HORIZ-9-PIN
Changed lines of the file:
@@
 F 0 "J1" H 800 2700 50  0000 C CNN
 F 1 "Screw_Terminal_01x09" H 800 2700 50  0001 C CNN
-F 2 "TerminalBlock_Phoenix:TerminalBlock_Phoenix_MKDS-3-9-5.08_1x09_P5.08mm_Horizontal" H 800 2200 50  0001 C CNN
+F 2 "PDJR-connectors:RS-PLUG-TERMINAL-HORIZ-9-PIN" H 800 2200 50  0001 C CNN
 F 3 "~" H 800 2200 50  0001 C CNN
 	1    800  2200
