File: hardware/kicad/opto_isolated_input.sch (KiCad schematic (older format))
At the start: 7 parts, among them Q1 BC547, Q2 BC337-40, U6 SFH617A-1

Commit message: SMD
Parts:
- D10: footprint Diode_THT:D_A-405_P2.54mm_Vertical_AnodeUp -> Diode_SMD:D_SOT-23_ANK
- Q1, Q2: footprint Package_TO_SOT_THT:TO-92_Inline -> Package_TO_SOT_SMD:TSOT-23
- R4, R5, R6: footprint Resistor_THT:R_Axial_DIN0207_L6.3mm_D2.5mm_P2.54mm_Vertical -> Resistor_SMD:R_0805_2012Metric
- U6: footprint Package_DIP:DIP-4_W7.62mm -> Package_DIP:SMDIP-4_W7.62mm
Changed lines of the file:
@@
 $Descr A4 11693 8268
 encoding utf-8
-Sheet 2 9
+Sheet 7 9
 Title "SIM108 Switch Input Module"
 Date "2022-06-11"
@@
 AR Path="/62F45EE0/62EBA913" Ref="U16"  Part="1"
 AR Path="/62FB890E/62EBA913" Ref="U18"  Part="1"
-F 0 "U20" H 6100 3200 50  0000 C CNN
+F 0 "U16" H 6100 3200 50  0000 C CNN
 F 1 "SFH617A-1" H 6100 3600 50  0000 C CNN
-F 2 "Package_DIP:DIP-4_W7.62mm" H 5900 3200 50  0001 L CIN
+F 2 "Package_DIP:SMDIP-4_W7.62mm" H 5900 3200 50  0001 L CIN
 F 3 "http://www.vishay.com/docs/83740/sfh617a.pdf" H 6100 3400 50  0001 L CNN
 	1    6100 3400
@@
 AR Path="/62F45EE0/62ED7963" Ref="R19"  Part="1"
 AR Path="/62FB890E/62ED7963" Ref="R22"  Part="1"
-F 0 "R25" H 5350 3500 50  0000 L CNN
+F 0 "R19" H 5350 3500 50  0000 L CNN
 F 1 "10K 0.5W" V 5300 3500 20  0000 C CNN
-F 2 "Resistor_THT:R_Axial_DIN0207_L6.3mm_D2.5mm_P2.54mm_Vertical" V 5230 3500 50  0001 C CNN
+F 2 "Resistor_SMD:R_0805_2012Metric" V 5230 3500 50  0001 C CNN
 F 3 "~" H 5300 3500 50  0001 C CNN
 F 4 "0.125W" V 5400 3500 50  0001 C CNN "Power"
@@
 AR Path="/62F45EE0/62F493CD" Ref="R20"  Part="1"
 AR Path="/62FB890E/62F493CD" Ref="R23"  Part="1"
-F 0 "R26" H 5750 4050 50  0000 L CNN
+F 0 "R20" H 5750 4050 50  0000 L CNN
 F 1 "100R 0.25W" V 5700 4050 20  0000 C CNN
-F 2 "Resistor_THT:R_Axial_DIN0207_L6.3mm_D2.5mm_P2.54mm_Vertical" V 5630 4050 50  0001 C CNN
+F 2 "Resistor_SMD:R_0805_2012Metric" V 5630 4050 50  0001 C CNN
 F 3 "~" H 5700 4050 50  0001 C CNN
 F 4 "0.125W" V 5800 4050 50  0001 C CNN "Power"
@@
 AR Path="/62F45EE0/62EA87F7" Ref="Q12"  Part="1"
 AR Path="/62FB890E/62EA87F7" Ref="Q14"  Part="1"
-F 0 "Q16" H 5791 3746 50  0000 L CNN
+F 0 "Q12" H 5791 3746 50  0000 L CNN
 F 1 "BC337-40" H 5791 3655 50  0000 L CNN
-F 2 "Package_TO_SOT_THT:TO-92_Inline" H 5800 3625 50  0001 L CIN
+F 2 "Package_TO_SOT_SMD:TSOT-23" H 5800 3625 50  0001 L CIN
 F 3 "https://diotec.com/tl_files/diotec/files/pdf/datasheets/bc337.pdf" H 5600 3700 50  0001 L CNN
 	1    5600 3700
@@
 AR Path="/62F45EE0/62FE9B9E" Ref="D15"  Part="1"
 AR Path="/62FB890E/62FE9B9E" Ref="D16"  Part="1"
-F 0 "D17" H 4750 3250 50  0000 L CNN
+F 0 "D15" H 4750 3250 50  0000 L CNN
 F 1 "IN4007" H 5000 3250 50  0000 L CNN
-F 2 "Diode_THT:D_A-405_P2.54mm_Vertical_AnodeUp" H 4950 3300 50  0001 C CNN
+F 2 "Diode_SMD:D_SOT-23_ANK" H 4950 3300 50  0001 C CNN
 F 3 "~" H 4950 3300 50  0001 C CNN
 F 4 "Y" H 4950 3300 50  0001 L CNN "Spice_Netlist_Enabled"
@@
 AR Path="/62F45EE0/62FB7374" Ref="Q11"  Part="1"
 AR Path="/62FB890E/62FB7374" Ref="Q13"  Part="1"
-F 0 "Q15" H 5591 3946 50  0000 L CNN
+F 0 "Q11" H 5591 3946 50  0000 L CNN
 F 1 "BC547" H 5591 3855 50  0000 L CNN
-F 2 "Package_TO_SOT_THT:TO-92_Inline" H 5600 3825 50  0001 L CIN
+F 2 "Package_TO_SOT_SMD:TSOT-23" H 5600 3825 50  0001 L CIN
 F 3 "https://www.onsemi.com/pub/Collateral/BC550-D.pdf" H 5400 3900 50  0001 L CNN
 	1    5400 3900
@@
 AR Path="/62F45EE0/6344909D" Ref="R21"  Part="1"
 AR Path="/62FB890E/6344909D" Ref="R24"  Part="1"
-F 0 "R27" H 6550 4050 50  0000 L CNN
+F 0 "R21" H 6550 4050 50  0000 L CNN
 F 1 "4K7 0.125W" V 6500 4050 20  0000 C CNN
-F 2 "Resistor_THT:R_Axial_DIN0207_L6.3mm_D2.5mm_P2.54mm_Vertical" V 6430 4050 50  0001 C CNN
+F 2 "Resistor_SMD:R_0805_2012Metric" V 6430 4050 50  0001 C CNN
 F 3 "~" H 6500 4050 50  0001 C CNN
 F 4 "0.125W" V 6600 4050 50  0001 C CNN "Power"

Commit message: Add test points
Changed lines of the file:
@@
 AR Path="/62F45EE0/62EBA913" Ref="U16"  Part="1"
 AR Path="/62FB890E/62EBA913" Ref="U18"  Part="1"
-F 0 "U16" H 6100 3200 50  0000 C CNN
+F 0 "U20" H 6100 3200 50  0000 C CNN
 F 1 "SFH617A-1" H 6100 3600 50  0000 C CNN
 F 2 "Package_DIP:SMDIP-4_W7.62mm" H 5900 3200 50  0001 L CIN
@@
 AR Path="/62F45EE0/62ED7963" Ref="R19"  Part="1"
 AR Path="/62FB890E/62ED7963" Ref="R22"  Part="1"
-F 0 "R19" H 5350 3500 50  0000 L CNN
+F 0 "R25" H 5350 3500 50  0000 L CNN
 F 1 "10K 0.5W" V 5300 3500 20  0000 C CNN
 F 2 "Resistor_SMD:R_0805_2012Metric" V 5230 3500 50  0001 C CNN
@@
 AR Path="/62F45EE0/62F493CD" Ref="R20"  Part="1"
 AR Path="/62FB890E/62F493CD" Ref="R23"  Part="1"
-F 0 "R20" H 5750 4050 50  0000 L CNN
+F 0 "R26" H 5750 4050 50  0000 L CNN
 F 1 "100R 0.25W" V 5700 4050 20  0000 C CNN
 F 2 "Resistor_SMD:R_0805_2012Metric" V 5630 4050 50  0001 C CNN
@@
 AR Path="/62F45EE0/62EA87F7" Ref="Q12"  Part="1"
 AR Path="/62FB890E/62EA87F7" Ref="Q14"  Part="1"
-F 0 "Q12" H 5791 3746 50  0000 L CNN
+F 0 "Q16" H 5791 3746 50  0000 L CNN
 F 1 "BC337-40" H 5791 3655 50  0000 L CNN
 F 2 "Package_TO_SOT_SMD:TSOT-23" H 5800 3625 50  0001 L CIN
@@
 AR Path="/62F45EE0/62FE9B9E" Ref="D15"  Part="1"
 AR Path="/62FB890E/62FE9B9E" Ref="D16"  Part="1"
-F 0 "D15" H 4750 3250 50  0000 L CNN
+F 0 "D17" H 4750 3250 50  0000 L CNN
 F 1 "IN4007" H 5000 3250 50  0000 L CNN
 F 2 "Diode_SMD:D_SOT-23_ANK" H 4950 3300 50  0001 C CNN
@@
 AR Path="/62F45EE0/62FB7374" Ref="Q11"  Part="1"
 AR Path="/62FB890E/62FB7374" Ref="Q13"  Part="1"
-F 0 "Q11" H 5591 3946 50  0000 L CNN
+F 0 "Q15" H 5591 3946 50  0000 L CNN
 F 1 "BC547" H 5591 3855 50  0000 L CNN
 F 2 "Package_TO_SOT_SMD:TSOT-23" H 5600 3825 50  0001 L CIN
@@
 AR Path="/62F45EE0/6344909D" Ref="R21"  Part="1"
 AR Path="/62FB890E/6344909D" Ref="R24"  Part="1"
-F 0 "R21" H 6550 4050 50  0000 L CNN
+F 0 "R27" H 6550 4050 50  0000 L CNN
 F 1 "4K7 0.125W" V 6500 4050 20  0000 C CNN
 F 2 "Resistor_SMD:R_0805_2012Metric" V 6430 4050 50  0001 C CNN

Commit message: Revise PCB
Connections:
- net OII_OUT: now also R6.2, U6.4; no longer R6.1, U6.3
- net OII_OUT_GND: now also U6.3; no longer R6.2
- net OII_OUT_VCC: now also R6.1; no longer U6.4
Other:
- moved on the sheet: R24
Changed lines of the file:
@@
 $Descr A4 11693 8268
 encoding utf-8
-Sheet 7 9
+Sheet 8 9
 Title "SIM108 Switch Input Module"
 Date "2022-06-11"
@@
 AR Path="/62F45EE0/62EBA913" Ref="U16"  Part="1"
 AR Path="/62FB890E/62EBA913" Ref="U18"  Part="1"
-F 0 "U20" H 6100 3200 50  0000 C CNN
+F 0 "U18" H 6100 3200 50  0000 C CNN
 F 1 "SFH617A-1" H 6100 3600 50  0000 C CNN
 F 2 "Package_DIP:SMDIP-4_W7.62mm" H 5900 3200 50  0001 L CIN
@@
 AR Path="/62F45EE0/62ED7963" Ref="R19"  Part="1"
 AR Path="/62FB890E/62ED7963" Ref="R22"  Part="1"
-F 0 "R25" H 5350 3500 50  0000 L CNN
+F 0 "R22" H 5350 3500 50  0000 L CNN
 F 1 "10K 0.5W" V 5300 3500 20  0000 C CNN
 F 2 "Resistor_SMD:R_0805_2012Metric" V 5230 3500 50  0001 C CNN
@@
 AR Path="/62F45EE0/62F493CD" Ref="R20"  Part="1"
 AR Path="/62FB890E/62F493CD" Ref="R23"  Part="1"
-F 0 "R26" H 5750 4050 50  0000 L CNN
+F 0 "R23" H 5750 4050 50  0000 L CNN
 F 1 "100R 0.25W" V 5700 4050 20  0000 C CNN
 F 2 "Resistor_SMD:R_0805_2012Metric" V 5630 4050 50  0001 C CNN
@@
 AR Path="/62F45EE0/62EA87F7" Ref="Q12"  Part="1"
 AR Path="/62FB890E/62EA87F7" Ref="Q14"  Part="1"
-F 0 "Q16" H 5791 3746 50  0000 L CNN
+F 0 "Q14" H 5791 3746 50  0000 L CNN
 F 1 "BC337-40" H 5791 3655 50  0000 L CNN
 F 2 "Package_TO_SOT_SMD:TSOT-23" H 5800 3625 50  0001 L CIN
@@
 AR Path="/62F45EE0/62FE9B9E" Ref="D15"  Part="1"
 AR Path="/62FB890E/62FE9B9E" Ref="D16"  Part="1"
-F 0 "D17" H 4750 3250 50  0000 L CNN
+F 0 "D16" H 4750 3250 50  0000 L CNN
 F 1 "IN4007" H 5000 3250 50  0000 L CNN
 F 2 "Diode_SMD:D_SOT-23_ANK" H 4950 3300 50  0001 C CNN
@@
 AR Path="/62F45EE0/62FB7374" Ref="Q11"  Part="1"
 AR Path="/62FB890E/62FB7374" Ref="Q13"  Part="1"
-F 0 "Q15" H 5591 3946 50  0000 L CNN
+F 0 "Q13" H 5591 3946 50  0000 L CNN
 F 1 "BC547" H 5591 3855 50  0000 L CNN
 F 2 "Package_TO_SOT_SMD:TSOT-23" H 5600 3825 50  0001 L CIN
@@
 Text HLabel 4750 4200 0    50   UnSpc ~ 0
 OII_IN_GND
-Text HLabel 7600 3500 2    50   Output ~ 0
+Text HLabel 7600 3300 2    50   Output ~ 0
 OII_OUT
 Text HLabel 7650 4200 2    50   UnSpc ~ 0
@@
 Wire Wire Line
 	6400 3300 6500 3300
-Wire Wire Line
-	6500 3300 6500 2800
 $Comp
 L Device:R R6
 U 1 1 6344909D
-P 6500 4050
+P 6500 3050
 AR Path="/62FB7846/6344909D" Ref="R6"  Part="1"
 AR Path="/63089671/6344909D" Ref="R27"  Part="1"
@@
 AR Path="/62F45EE0/6344909D" Ref="R21"  Part="1"
 AR Path="/62FB890E/6344909D" Ref="R24"  Part="1"
-F 0 "R27" H 6550 4050 50  0000 L CNN
-F 1 "4K7 0.125W" V 6500 4050 20  0000 C CNN
-F 2 "Resistor_SMD:R_0805_2012Metric" V 6430 4050 50  0001 C CNN
-F 3 "~" H 6500 4050 50  0001 C CNN
-F 4 "0.125W" V 6600 4050 50  0001 C CNN "Power"
-	1    6500 4050
-	1    0    0    -1
-$EndComp
-Wire Wire Line
-	6500 3900 6500 3500
-Connection ~ 6500 3500
+F 0 "R24" H 6550 3050 50  0000 L CNN
+F 1 "4K7 0.125W" V 6500 3050 20  0000 C CNN
+F 2 "Resistor_SMD:R_0805_2012Metric" V 6430 3050 50  0001 C CNN
+F 3 "~" H 6500 3050 50  0001 C CNN
+F 4 "0.125W" V 6600 3050 50  0001 C CNN "Power"
+	1    6500 3050
+	1    0    0    -1
+$EndComp
+Wire Wire Line
+	6500 4200 6500 3500
 Wire Wire Line
 	4750 4200 5300 4200
@@
 	6500 4200 7650 4200
 Wire Wire Line
-	6500 3500 7600 3500
+	6500 2900 6500 2800
+Wire Wire Line
+	6500 3300 6500 3200
+Wire Wire Line
+	6500 3300 7600 3300
+Connection ~ 6500 3300
 $EndSCHEMATC

Commit message: Edit silk.
Changed lines of the file:
@@
 $Descr A4 11693 8268
 encoding utf-8
-Sheet 8 9
+Sheet 2 9
 Title "SIM108 Switch Input Module"
 Date "2022-06-11"
@@
 AR Path="/62F45EE0/62EBA913" Ref="U16"  Part="1"
 AR Path="/62FB890E/62EBA913" Ref="U18"  Part="1"
-F 0 "U18" H 6100 3200 50  0000 C CNN
+F 0 "U6" H 6100 3200 50  0000 C CNN
 F 1 "SFH617A-1" H 6100 3600 50  0000 C CNN
 F 2 "Package_DIP:SMDIP-4_W7.62mm" H 5900 3200 50  0001 L CIN
@@
 AR Path="/62F45EE0/62ED7963" Ref="R19"  Part="1"
 AR Path="/62FB890E/62ED7963" Ref="R22"  Part="1"
-F 0 "R22" H 5350 3500 50  0000 L CNN
+F 0 "R4" H 5350 3500 50  0000 L CNN
 F 1 "10K 0.5W" V 5300 3500 20  0000 C CNN
 F 2 "Resistor_SMD:R_0805_2012Metric" V 5230 3500 50  0001 C CNN
@@
 AR Path="/62F45EE0/62F493CD" Ref="R20"  Part="1"
 AR Path="/62FB890E/62F493CD" Ref="R23"  Part="1"
-F 0 "R23" H 5750 4050 50  0000 L CNN
+F 0 "R5" H 5750 4050 50  0000 L CNN
 F 1 "100R 0.25W" V 5700 4050 20  0000 C CNN
 F 2 "Resistor_SMD:R_0805_2012Metric" V 5630 4050 50  0001 C CNN
@@
 AR Path="/62F45EE0/62EA87F7" Ref="Q12"  Part="1"
 AR Path="/62FB890E/62EA87F7" Ref="Q14"  Part="1"
-F 0 "Q14" H 5791 3746 50  0000 L CNN
+F 0 "Q2" H 5791 3746 50  0000 L CNN
 F 1 "BC337-40" H 5791 3655 50  0000 L CNN
 F 2 "Package_TO_SOT_SMD:TSOT-23" H 5800 3625 50  0001 L CIN
@@
 AR Path="/62F45EE0/62FE9B9E" Ref="D15"  Part="1"
 AR Path="/62FB890E/62FE9B9E" Ref="D16"  Part="1"
-F 0 "D16" H 4750 3250 50  0000 L CNN
+F 0 "D10" H 4750 3250 50  0000 L CNN
 F 1 "IN4007" H 5000 3250 50  0000 L CNN
 F 2 "Diode_SMD:D_SOT-23_ANK" H 4950 3300 50  0001 C CNN
@@
 AR Path="/62F45EE0/62FB7374" Ref="Q11"  Part="1"
 AR Path="/62FB890E/62FB7374" Ref="Q13"  Part="1"
-F 0 "Q13" H 5591 3946 50  0000 L CNN
+F 0 "Q1" H 5591 3946 50  0000 L CNN
 F 1 "BC547" H 5591 3855 50  0000 L CNN
 F 2 "Package_TO_SOT_SMD:TSOT-23" H 5600 3825 50  0001 L CIN
@@
 AR Path="/62F45EE0/6344909D" Ref="R21"  Part="1"
 AR Path="/62FB890E/6344909D" Ref="R24"  Part="1"
-F 0 "R24" H 6550 3050 50  0000 L CNN
+F 0 "R6" H 6550 3050 50  0000 L CNN
 F 1 "4K7 0.125W" V 6500 3050 20  0000 C CNN
 F 2 "Resistor_SMD:R_0805_2012Metric" V 6430 3050 50  0001 C CNN
