File: hardware/kicad/PDJRSIM.kicad_pcb (KiCad board)
At the start: 2 copper layers, 100 x 85 mm, 110 parts, among them J1 Screw_Terminal_01x09, J101 CAN, J2 Screw_Terminal_01x09, Q101 BSS138, Q102 BSS138, SW101 BUS, SW102 ADDR/VALUE, SW103 PRG, U1 BCR401, U10 BCR401 (16x)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

Commit message: Fix a break
Parts:
- U10, U11, U12, U13, U15, U16, U18, U19, U21, U22, U5, U7, U8: value BCR401 (16x) -> BCR401
