File: hardware/kicad/PDJRSIM.sch (KiCad schematic (older format))
At the start: 54 parts, among them J1 Screw_Terminal_01x09, J2 Screw_Terminal_01x09, U1 BCR401, U10 BCR401 (16x), U11 BCR401 (16x), U12 BCR401 (16x), U13 BCR401 (16x), U14 ASCL-6400, U15 BCR401 (16x), U16 BCR401 (16x)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

Commit message: Rename
Parts:
- removed U1, U4: BCR401, PDJR_Connectors:BCR401, symbol SIM108-rescue:BCR401-pdjr
- removed U10, U11, U12, U13, U15, U16, U18, U19, U21, U22, U5, U7, U8: BCR401 (16x), PDJR_Connectors:BCR401, symbol SIM108-rescue:BCR401-pdjr
- U2: symbol SIM108-rescue:BCR401-pdjr -> PDJRSIM-rescue:BCR401-pdjr
Connections:
- net labels added: D22
Changed lines of the file:
@@
 encoding utf-8
 Sheet 1 1
-Title "SIM108 Switch Input Module"
+TiPDJRSIM Switch Input Module"
 Date "2022-06-11"
 Rev "2.0.0"
@@
 	1000 5100 1100 5100
 $Comp
-L SIM108-rescue:BCR401-pdjr U2
+L PDJRSIM-rescue:BCR401-pdjr U2
 U 1 1 644E29F9
 P 1550 4350
@@
 	0    -1   -1   0
 $EndComp
-$Comp
-L SIM108-rescue:BCR401-pdjr U4
+$CoPDJRSIM-rescue:BCR401-pdjr U4
 U 1 1 644E484A
 P 1750 4350
@@
 	0    -1   -1   0
 $EndComp
-$Comp
-L SIM108-rescue:BCR401-pdjr U1
+$CoPDJRSIM-rescue:BCR401-pdjr U1
 U 1 1 644E5BAF
 P 1350 4350
@@
 	0    -1   -1   0
 $EndComp
-$Comp
-L SIM108-rescue:BCR401-pdjr U5
+$CoPDJRSIM-rescue:BCR401-pdjr U5
 U 1 1 644E608B
 P 1950 4350
@@
 Wire Wire Line
 	2150 4800 3500 4800
-$Comp
-L SIM108-rescue:BCR401-pdjr U8
+$CoPDJRSIM-rescue:BCR401-pdjr U8
 U 1 1 647CB8BF
 P 4750 4350
@@
 	0    -1   -1   0
 $EndComp
-$Comp
-L SIM108-rescue:BCR401-pdjr U7
+$CoPDJRSIM-rescue:BCR401-pdjr U7
 U 1 1 647CD502
 P 4550 4350
@@
 	0    -1   -1   0
 $EndComp
-$Comp
-L SIM108-rescue:BCR401-pdjr U10
+$CoPDJRSIM-rescue:BCR401-pdjr U10
 U 1 1 64838AC9
 P 4950 4350
@@
 	0    -1   -1   0
 $EndComp
-$Comp
-L SIM108-rescue:BCR401-pdjr U11
+$CoPDJRSIM-rescue:BCR401-pdjr U11
 U 1 1 648391A6
 P 5150 4350
@@
 	0    -1   -1   0
 $EndComp
-$Comp
-L SIM108-rescue:BCR401-pdjr U12
+$CoPDJRSIM-rescue:BCR401-pdjr U12
 U 1 1 6483971E
 P 6300 4350
@@
 	0    -1   -1   0
 $EndComp
-$Comp
-L SIM108-rescue:BCR401-pdjr U13
+$CoPDJRSIM-rescue:BCR401-pdjr U13
 U 1 1 6483A429
 P 6500 4350
@@
 	0    -1   -1   0
 $EndComp
-$Comp
-L SIM108-rescue:BCR401-pdjr U15
+$CoPDJRSIM-rescue:BCR401-pdjr U15
 U 1 1 6483AAD4
 P 6700 4350
@@
 	0    -1   -1   0
 $EndComp
-$Comp
-L SIM108-rescue:BCR401-pdjr U16
+$CoPDJRSIM-rescue:BCR401-pdjr U16
 U 1 1 6483AF5A
 P 6900 4350
@@
 	0    -1   -1   0
 $EndComp
-$Comp
-L SIM108-rescue:BCR401-pdjr U18
+$CoPDJRSIM-rescue:BCR401-pdjr U18
 U 1 1 6483B5AA
 P 9500 4350
@@
 	0    -1   -1   0
 $EndComp
-$Comp
-L SIM108-rescue:BCR401-pdjr U19
+$CoPDJRSIM-rescue:BCR401-pdjr U19
 U 1 1 6483C163
 P 9700 4350
@@
 	0    -1   -1   0
 $EndComp
-$Comp
-L SIM108-rescue:BCR401-pdjr U21
+$CoPDJRSIM-rescue:BCR401-pdjr U21
 U 1 1 6483C5F7
 P 9900 4350
@@
 	0    -1   -1   0
 $EndComp
-$Comp
-L SIM108-rescue:BCR401-pdjr U22
+$CoPDJRSIM-rescue:BCR401-pdjr U22
 U 1 1 6483CA64
 P 10100 4350
@@
 Wire Wire Line
 	1300 6400 10200 6400
+Text Label 10450 850  0    50   ~ 0
+D22
 $EndSCHEMATC

Commit message: Fix a break
Parts:
- added U1, U10, U11, U12, U13, U15, U16, U18, U19, U21, U22, U4, U5, U7, U8: BCR401, PDJR_Connectors:BCR401, symbol PDJRSIM-rescue:BCR401-pdjr
Connections:
- net labels removed: D22
Changed lines of the file:
@@
 encoding utf-8
 Sheet 1 1
-TiPDJRSIM Switch Input Module"
+Title ""
 Date "2022-06-11"
 Rev "2.0.0"
@@
 	0    -1   -1   0
 $EndComp
-$CoPDJRSIM-rescue:BCR401-pdjr U4
-U 1 1 644E484A
-P 1750 4350
-F 0 "U4" V 2000 4200 50  0000 R CNN
-F 1 "BCR401" V 1705 4072 50  0001 R CNN
-F 2 "PDJR_Connectors:BCR401" H 1250 3850 50  0001 C CNN
-F 3 "" H 1250 3850 50  0001 C CNN
-	1    1750 4350
-	0    -1   -1   0
-$EndComp
-$CoPDJRSIM-rescue:BCR401-pdjr U1
-U 1 1 644E5BAF
-P 1350 4350
-F 0 "U1" V 1600 4200 50  0000 R CNN
-F 1 "BCR401" V 1305 4072 50  0001 R CNN
-F 2 "PDJR_Connectors:BCR401" H 850 3850 50  0001 C CNN
-F 3 "" H 850 3850 50  0001 C CNN
-	1    1350 4350
-	0    -1   -1   0
-$EndComp
-$CoPDJRSIM-rescue:BCR401-pdjr U5
-U 1 1 644E608B
-P 1950 4350
-F 0 "U5" V 2200 4200 50  0000 R CNN
-F 1 "BCR401 (16x)" V 1905 4072 50  0000 R CNN
-F 2 "PDJR_Connectors:BCR401" H 1450 3850 50  0001 C CNN
-F 3 "" H 1450 3850 50  0001 C CNN
-	1    1950 4350
-	0    -1   -1   0
-$EndComp
 Wire Wire Line
 	2100 4050 2100 3900
@@
 Wire Wire Line
 	2150 4800 3500 4800
-$CoPDJRSIM-rescue:BCR401-pdjr U8
-U 1 1 647CB8BF
-P 4750 4350
-F 0 "U8" V 5000 4200 50  0000 R CNN
-F 1 "BCR401 (16x)" V 4705 4072 50  0001 R CNN
-F 2 "PDJR_Connectors:BCR401" H 4250 3850 50  0001 C CNN
-F 3 "" H 4250 3850 50  0001 C CNN
-	1    4750 4350
-	0    -1   -1   0
-$EndComp
-$CoPDJRSIM-rescue:BCR401-pdjr U7
-U 1 1 647CD502
-P 4550 4350
-F 0 "U7" V 4800 4200 50  0000 R CNN
-F 1 "BCR401 (16x)" V 4505 4072 50  0001 R CNN
-F 2 "PDJR_Connectors:BCR401" H 4050 3850 50  0001 C CNN
-F 3 "" H 4050 3850 50  0001 C CNN
-	1    4550 4350
-	0    -1   -1   0
-$EndComp
-$CoPDJRSIM-rescue:BCR401-pdjr U10
-U 1 1 64838AC9
-P 4950 4350
-F 0 "U10" V 5200 4200 50  0000 R CNN
-F 1 "BCR401 (16x)" V 4905 4072 50  0001 R CNN
-F 2 "PDJR_Connectors:BCR401" H 4450 3850 50  0001 C CNN
-F 3 "" H 4450 3850 50  0001 C CNN
-	1    4950 4350
-	0    -1   -1   0
-$EndComp
-$CoPDJRSIM-rescue:BCR401-pdjr U11
-U 1 1 648391A6
-P 5150 4350
-F 0 "U11" V 5400 4200 50  0000 R CNN
-F 1 "BCR401 (16x)" V 5105 4072 50  0001 R CNN
-F 2 "PDJR_Connectors:BCR401" H 4650 3850 50  0001 C CNN
-F 3 "" H 4650 3850 50  0001 C CNN
-	1    5150 4350
-	0    -1   -1   0
-$EndComp
-$CoPDJRSIM-rescue:BCR401-pdjr U12
-U 1 1 6483971E
-P 6300 4350
-F 0 "U12" V 6550 4200 50  0000 R CNN
-F 1 "BCR401 (16x)" V 6255 4072 50  0001 R CNN
-F 2 "PDJR_Connectors:BCR401" H 5800 3850 50  0001 C CNN
-F 3 "" H 5800 3850 50  0001 C CNN
-	1    6300 4350
-	0    -1   -1   0
-$EndComp
-$CoPDJRSIM-rescue:BCR401-pdjr U13
-U 1 1 6483A429
-P 6500 4350
-F 0 "U13" V 6750 4200 50  0000 R CNN
-F 1 "BCR401 (16x)" V 6455 4072 50  0001 R CNN
-F 2 "PDJR_Connectors:BCR401" H 6000 3850 50  0001 C CNN
-F 3 "" H 6000 3850 50  0001 C CNN
-	1    6500 4350
-	0    -1   -1   0
-$EndComp
-$CoPDJRSIM-rescue:BCR401-pdjr U15
-U 1 1 6483AAD4
-P 6700 4350
-F 0 "U15" V 6950 4200 50  0000 R CNN
-F 1 "BCR401 (16x)" V 6655 4072 50  0001 R CNN
-F 2 "PDJR_Connectors:BCR401" H 6200 3850 50  0001 C CNN
-F 3 "" H 6200 3850 50  0001 C CNN
-	1    6700 4350
-	0    -1   -1   0
-$EndComp
-$CoPDJRSIM-rescue:BCR401-pdjr U16
-U 1 1 6483AF5A
-P 6900 4350
-F 0 "U16" V 7150 4200 50  0000 R CNN
-F 1 "BCR401 (16x)" V 6855 4072 50  0001 R CNN
-F 2 "PDJR_Connectors:BCR401" H 6400 3850 50  0001 C CNN
-F 3 "" H 6400 3850 50  0001 C CNN
-	1    6900 4350
-	0    -1   -1   0
-$EndComp
-$CoPDJRSIM-rescue:BCR401-pdjr U18
-U 1 1 6483B5AA
-P 9500 4350
-F 0 "U18" V 9750 4200 50  0000 R CNN
-F 1 "BCR401 (16x)" V 9455 4072 50  0001 R CNN
-F 2 "PDJR_Connectors:BCR401" H 9000 3850 50  0001 C CNN
-F 3 "" H 9000 3850 50  0001 C CNN
-	1    9500 4350
-	0    -1   -1   0
-$EndComp
-$CoPDJRSIM-rescue:BCR401-pdjr U19
-U 1 1 6483C163
-P 9700 4350
-F 0 "U19" V 9950 4200 50  0000 R CNN
-F 1 "BCR401 (16x)" V 9655 4072 50  0001 R CNN
-F 2 "PDJR_Connectors:BCR401" H 9200 3850 50  0001 C CNN
-F 3 "" H 9200 3850 50  0001 C CNN
-	1    9700 4350
-	0    -1   -1   0
-$EndComp
-$CoPDJRSIM-rescue:BCR401-pdjr U21
-U 1 1 6483C5F7
-P 9900 4350
-F 0 "U21" V 10150 4200 50  0000 R CNN
-F 1 "BCR401 (16x)" V 9855 4072 50  0001 R CNN
-F 2 "PDJR_Connectors:BCR401" H 9400 3850 50  0001 C CNN
-F 3 "" H 9400 3850 50  0001 C CNN
-	1    9900 4350
-	0    -1   -1   0
-$EndComp
-$CoPDJRSIM-rescue:BCR401-pdjr U22
-U 1 1 6483CA64
-P 10100 4350
-F 0 "U22" V 10350 4200 50  0000 R CNN
-F 1 "BCR401 (16x)" V 10055 4072 50  0001 R CNN
-F 2 "PDJR_Connectors:BCR401" H 9600 3850 50  0001 C CNN
-F 3 "" H 9600 3850 50  0001 C CNN
-	1    10100 4350
-	0    -1   -1   0
-$EndComp
 Wire Wire Line
 	4700 3900 4700 4050
@@
 Wire Wire Line
 	1300 6400 10200 6400
-Text Label 10450 850  0    50   ~ 0
-D22
+$Comp
+L PDJRSIM-rescue:BCR401-pdjr U1
+U 1 1 63E7712E
+P 1350 4350
+F 0 "U1" V 1600 4200 50  0000 R CNN
+F 1 "BCR401" V 1305 4072 50  0001 R CNN
+F 2 "PDJR_Connectors:BCR401" H 850 3850 50  0001 C CNN
+F 3 "" H 850 3850 50  0001 C CNN
+	1    1350 4350
+	0    -1   -1   0
+$EndComp
+$Comp
+L PDJRSIM-rescue:BCR401-pdjr U4
+U 1 1 63E778F7
+P 1750 4350
+F 0 "U4" V 2000 4200 50  0000 R CNN
+F 1 "BCR401" V 1705 4072 50  0001 R CNN
+F 2 "PDJR_Connectors:BCR401" H 1250 3850 50  0001 C CNN
+F 3 "" H 1250 3850 50  0001 C CNN
+	1    1750 4350
+	0    -1   -1   0
+$EndComp
+$Comp
+L PDJRSIM-rescue:BCR401-pdjr U5
+U 1 1 63E77DD9
+P 1950 4350
+F 0 "U5" V 2200 4200 50  0000 R CNN
+F 1 "BCR401" V 1905 4072 50  0001 R CNN
+F 2 "PDJR_Connectors:BCR401" H 1450 3850 50  0001 C CNN
+F 3 "" H 1450 3850 50  0001 C CNN
+	1    1950 4350
+	0    -1   -1   0
+$EndComp
+$Comp
+L PDJRSIM-rescue:BCR401-pdjr U7
+U 1 1 63E78162
+P 4550 4350
+F 0 "U7" V 4800 4200 50  0000 R CNN
+F 1 "BCR401" V 4505 4072 50  0001 R CNN
+F 2 "PDJR_Connectors:BCR401" H 4050 3850 50  0001 C CNN
+F 3 "" H 4050 3850 50  0001 C CNN
+	1    4550 4350
+	0    -1   -1   0
+$EndComp
+$Comp
+L PDJRSIM-rescue:BCR401-pdjr U8
+U 1 1 63E79999
+P 4750 4350
+F 0 "U8" V 5000 4200 50  0000 R CNN
+F 1 "BCR401" V 4705 4072 50  0001 R CNN
+F 2 "PDJR_Connectors:BCR401" H 4250 3850 50  0001 C CNN
+F 3 "" H 4250 3850 50  0001 C CNN
+	1    4750 4350
+	0    -1   -1   0
+$EndComp
+$Comp
+L PDJRSIM-rescue:BCR401-pdjr U10
+U 1 1 63E79EF0
+P 4950 4350
+F 0 "U10" V 5200 4200 50  0000 R CNN
+F 1 "BCR401" V 4905 4072 50  0001 R CNN
+F 2 "PDJR_Connectors:BCR401" H 4450 3850 50  0001 C CNN
+F 3 "" H 4450 3850 50  0001 C CNN
+	1    4950 4350
+	0    -1   -1   0
+$EndComp
+$Comp
+L PDJRSIM-rescue:BCR401-pdjr U11
+U 1 1 63E7A3B5
+P 5150 4350
+F 0 "U11" V 5400 4200 50  0000 R CNN
+F 1 "BCR401" V 5105 4072 50  0001 R CNN
+F 2 "PDJR_Connectors:BCR401" H 4650 3850 50  0001 C CNN
+F 3 "" H 4650 3850 50  0001 C CNN
+	1    5150 4350
+	0    -1   -1   0
+$EndComp
+$Comp
+L PDJRSIM-rescue:BCR401-pdjr U12
+U 1 1 63E7A8A6
+P 6300 4350
+F 0 "U12" V 6550 4200 50  0000 R CNN
+F 1 "BCR401" V 6255 4072 50  0001 R CNN
+F 2 "PDJR_Connectors:BCR401" H 5800 3850 50  0001 C CNN
+F 3 "" H 5800 3850 50  0001 C CNN
+	1    6300 4350
+	0    -1   -1   0
+$EndComp
+$Comp
+L PDJRSIM-rescue:BCR401-pdjr U13
+U 1 1 63E7AE37
+P 6500 4350
+F 0 "U13" V 6750 4200 50  0000 R CNN
+F 1 "BCR401" V 6455 4072 50  0001 R CNN
+F 2 "PDJR_Connectors:BCR401" H 6000 3850 50  0001 C CNN
+F 3 "" H 6000 3850 50  0001 C CNN
+	1    6500 4350
+	0    -1   -1   0
+$EndComp
+$Comp
+L PDJRSIM-rescue:BCR401-pdjr U15
+U 1 1 63E7B2F1
+P 6700 4350
+F 0 "U15" V 6950 4200 50  0000 R CNN
+F 1 "BCR401" V 6655 4072 50  0001 R CNN
+F 2 "PDJR_Connectors:BCR401" H 6200 3850 50  0001 C CNN
+F 3 "" H 6200 3850 50  0001 C CNN
+	1    6700 4350
+	0    -1   -1   0
+$EndComp
+$Comp
+L PDJRSIM-rescue:BCR401-pdjr U16
+U 1 1 63E7B87C
+P 6900 4350
+F 0 "U16" V 7150 4200 50  0000 R CNN
+F 1 "BCR401" V 6855 4072 50  0001 R CNN
+F 2 "PDJR_Connectors:BCR401" H 6400 3850 50  0001 C CNN
+F 3 "" H 6400 3850 50  0001 C CNN
+	1    6900 4350
+	0    -1   -1   0
+$EndComp
+$Comp
+L PDJRSIM-rescue:BCR401-pdjr U18
+U 1 1 63E7BC35
+P 9500 4350
+F 0 "U18" V 9750 4200 50  0000 R CNN
+F 1 "BCR401" V 9455 4072 50  0001 R CNN
+F 2 "PDJR_Connectors:BCR401" H 9000 3850 50  0001 C CNN
+F 3 "" H 9000 3850 50  0001 C CNN
+	1    9500 4350
+	0    -1   -1   0
+$EndComp
+$Comp
+L PDJRSIM-rescue:BCR401-pdjr U19
+U 1 1 63E7D026
+P 9700 4350
+F 0 "U19" V 9950 4200 50  0000 R CNN
+F 1 "BCR401" V 9655 4072 50  0001 R CNN
+F 2 "PDJR_Connectors:BCR401" H 9200 3850 50  0001 C CNN
+F 3 "" H 9200 3850 50  0001 C CNN
+	1    9700 4350
+	0    -1   -1   0
+$EndComp
+$Comp
+L PDJRSIM-rescue:BCR401-pdjr U21
+U 1 1 63E7D429
+P 9900 4350
+F 0 "U21" V 10150 4200 50  0000 R CNN
+F 1 "BCR401" V 9855 4072 50  0001 R CNN
+F 2 "PDJR_Connectors:BCR401" H 9400 3850 50  0001 C CNN
+F 3 "" H 9400 3850 50  0001 C CNN
+	1    9900 4350
+	0    -1   -1   0
+$EndComp
+$Comp
+L PDJRSIM-rescue:BCR401-pdjr U22
+U 1 1 63E7D870
+P 10100 4350
+F 0 "U22" V 10350 4200 50  0000 R CNN
+F 1 "BCR401" V 10055 4072 50  0001 R CNN
+F 2 "PDJR_Connectors:BCR401" H 9600 3850 50  0001 C CNN
+F 3 "" H 9600 3850 50  0001 C CNN
+	1    10100 4350
+	0    -1   -1   0
+$EndComp
 $EndSCHEMATC
